File: hardware/trans-led-board/trans-led-board.kicad_pcb (KiCad board)
At the start: 2 copper layers, 12 x 33 mm, 5 parts, among them J1 Conn_01x02

Commit message: Updated transmission LED footprint and added fiducials
Parts:
- added FID1: Fiducial, Fiducial:Fiducial_1mm_Mask2mm, F.Cu at (115.8, 88.0)
- added FID2: Fiducial, Fiducial:Fiducial_1mm_Mask2mm, F.Cu at (115.8, 59.0)
- added FID3: Fiducial, Fiducial:Fiducial_1mm_Mask2mm, F.Cu at (124.2, 59.0)
Other:
- board text added: "Rev: C* 2021-??-??"
- board text removed: "Rev: B 2021-10-06"

Commit message: Update schematic properties
Changed all revision labeling to "C" with today's date. This is subject
to change when the boards are sent for manufacturing, but removing
placeholders make mistakes here less likely in the future.

Set grid and drill origins to what they're hopefully supposed to be. Not
sure how much this matters, but it probably won't hurt.

More layout nitpicking and review changes may happen between now and
pre-production, but the general design and layout for Rev C can
probably be considered sufficiently done for now.
Other:
- board text added: "Rev: C 2021-11-30"
- board text removed: "Rev: C* 2021-??-??"

Commit message: Migrate project from KiCad v5 to v6
- Update symbol library files for KiCad 6
- Moved location of symbol datasheet elements, since v6 suddenly decided
  they should always be visible in the symbol editor
- Update transmission LED board for KiCad 6
  - No real changes needed here, just the automated conversion and cleanup
  - Also adjusted silkscreen rev/date fields to use variables
- Update main board for KiCad 6
  - Fixed symbol and 3D model associations where necessary
  - Ran automated housekeeping fixups
  - Adjusted silkscreen rev/date fields to use variables
- Made changes to main board PCB to make DRC happy
  - Made minor tweaks to DRC rules based on fab specs
  - Tweaked footprint courtyard on net ties to fix violations, as these
    "components" only exist to make schematic ERC happy and might as
    well just be ordinary traces otherwise.
  - Tweaked silkscreen on USB connector to fix overhang violations
  - Modified traces around boot0 button, TC footprint, and USB
    connector, to avoid hole-to-trace clearance violations.

Scripted/configured panelization still needs work, and its unclear if
its KiKit issues or usage issues. It can generate the output, but needs
some nudging to get past build errors.

The USB connector should probably get another pass at routing, so the
VBUS and CC lines are a bit cleaner in implementation now.

Fix #24
Other:
- net class Default removed
- board text added: "Rev: ${REVISION} ${ISSUE_DATE}"
- board text removed: "Rev: C 2021-11-30"
