File: hardware/trans-led-board/trans-led-board.kicad_sch (KiCad schematic)
At the start: 7 parts, among them J1 Conn_01x02

Commit message: Update schematic BOM data based on actual parts ordered
Several components have changed suppliers and/or manufacturers between
the initial design prototypes and the bulk component orders. This
changes BOM data to reflect that.
Parts:
- D1: Supplier Digi-Key -> Mouser; Supplier PN 732-5666-1-ND -> 710-158302250
- J1: Supplier TLC -> Newark; Supplier PN SM02B-SRSS-TB(LF)(SN) -> 33P8179
Changed lines of the file:
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@@
       (effects (font (size 1.27 1.27)) hide)
     )
-    (property "Supplier" "Digi-Key" (id 7) (at 73.66 55.88 0)
+    (property "Supplier" "Mouser" (id 7) (at 73.66 55.88 0)
       (effects (font (size 1.27 1.27)) hide)
     )
-    (property "Supplier PN" "732-5666-1-ND" (id 8) (at 73.66 55.88 0)
+    (property "Supplier PN" "710-158302250" (id 8) (at 73.66 55.88 0)
       (effects (font (size 1.27 1.27)) hide)
     )
@@
       (effects (font (size 1.27 1.27)) hide)
     )
-    (property "Supplier" "TLC" (id 7) (at 58.42 53.34 0)
+    (property "Supplier" "Newark" (id 7) (at 58.42 53.34 0)
       (effects (font (size 1.27 1.27)) hide)
     )
-    (property "Supplier PN" "SM02B-SRSS-TB(LF)(SN)" (id 8) (at 58.42 53.34 0)
+    (property "Supplier PN" "33P8179" (id 8) (at 58.42 53.34 0)
       (effects (font (size 1.27 1.27)) hide)
     )

Commit message: Update metadata for schematic for LED symbol to make ERC happy
KiCad has changed the name of this symbol in the library, so we should
adjust the reference.

This isn't a real change to the schematic or PCB, just a library
reference tweak.
Parts:
- D1: symbol Device:LED_ALT -> Device:LED_Filled
Changed lines of the file:
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@@
     (effects (font (size 1.27 1.27)) (justify left bottom))
   )
-  (symbol (lib_id "Device:LED_ALT") (at 73.66 55.88 0) (unit 1)
+  (symbol (lib_id "Device:LED_Filled") (at 73.66 55.88 0) (unit 1)
     (in_bom yes) (on_board yes)
     (property "Reference" "D1" (id 0) (at 73.66 52.705 0))
