File: hardware/main-board/main-board.kicad_sch (KiCad schematic)
At the start: 87 parts, among them J1 USB_C_Receptacle_USB2.0, J2 DNI, J3 Display Connector, J4 Conn_01x02, SW1 SW_Push, SW2 SW_Push, SW3 SW_Push, SW4 SW_Push, SW5 SW_Detect, SW6 SW_Boot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

Commit message: Various panel related adjustments
Changed tab settings and positions for better size and component
clearance.
Nudged some traces around.
Parts:
- TP1: now left out of the parts list
Changed lines of the file:
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@@
   )
   (symbol (lib_id "Connector:TestPoint") (at 173.99 161.925 0) (unit 1)
-    (in_bom yes) (on_board yes)
+    (in_bom no) (on_board yes)
     (property "Reference" "TP1" (id 0) (at 175.4632 160.0962 0)
       (effects (font (size 1.27 1.27)) (justify left))
